File: New Version/Cheetah Driver Integrated V4 connector/HKCV4.brd (EAGLE design)
At the start: 49.5 x 37 mm, 72 parts, among them Q1 TPH, Q2 TPH, Q3 TPH, Q4 TPH, Q5 TPH, Q6 TPH

Commit message: updated can connector to harwin high-reliability latching
Parts:
- removed CAN: 5267-3, con-molex-spox:5267-3
- added U$8: 3-PIN, Ben_Library:M80-8430342
Connections:
- net CANH: now also U$8.2; no longer CAN.P$2
- net CANL: now also U$8.1; no longer CAN.P$1
- net GND: now also U$8.3; no longer CAN.P$3
Routing:
- net GND: track 139.8 -> 137.9 mm
Changed lines of the file:
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@@
 <layer number="24" name="bOrigins" color="15" fill="1" visible="yes" active="yes"/>
 <layer number="25" name="tNames" color="7" fill="1" visible="yes" active="yes"/>
-<layer number="26" name="bNames" color="7" fill="1" visible="no" active="yes"/>
+<layer number="26" name="bNames" color="7" fill="1" visible="yes" active="yes"/>
 <layer number="27" name="tValues" color="7" fill="1" visible="no" active="yes"/>
 <layer number="28" name="bValues" color="7" fill="1" visible="no" active="yes"/>
@@
 </element>
 <element name="U$9" library="Ben_Library" package="XT30_HORIZONTAL" value="XT30" x="17.76" y="-5.12" rot="MR90"/>
-<element name="CAN" library="con-molex-spox" package="5267-3" value="5267-3" x="24.4" y="4" smashed="yes" rot="MR90">
-<attribute name="NAME" x="19.74" y="4.46" size="1.27" layer="22" rot="MR90"/>
-</element>
 <element name="C21" library="rcl" package="C1206K" value="10 uF 50v" x="27.25" y="-4" smashed="yes">
 <attribute name="VALUE" x="25.65" y="-6.1" size="1.016" layer="27"/>
@@
 <attribute name="VALUE" x="25.65" y="-10.6" size="1.016" layer="27"/>
 </element>
+<element name="U$8" library="Ben_Library" package="M80-8430342" value="3-PIN" x="24.6" y="6.45" rot="MR270"/>
 </elements>
 <signals>
@@
 <wire x1="-0.76" y1="13.505" x2="-0.887" y2="13.505" width="0.16" layer="1"/>
 <wire x1="-0.887" y1="13.505" x2="-0.887" y2="11.41" width="0.16" layer="1"/>
-<contactref element="CAN" pad="P$3"/>
 <contactref element="U$9" pad="-"/>
 <polygon width="0.254" layer="16" isolate="0.254" thermals="no" rank="2">
@@
 <vertex x="14" y="-1"/>
 </polygon>
-<wire x1="24.4" y1="9" x2="23.5" y2="9" width="0.16" layer="3"/>
-<wire x1="23.5" y1="9" x2="18.5" y2="4" width="0.16" layer="3"/>
 <contactref element="C21" pad="2"/>
 <contactref element="C22" pad="2"/>
@@
 <via x="27.75" y="-3.5" extent="1-16" drill="0.3"/>
 <via x="27.75" y="-4.7" extent="1-16" drill="0.3"/>
+<contactref element="U$8" pad="3"/>
+<wire x1="24.6" y1="8.45" x2="18.8" y2="8.45" width="0.16" layer="3"/>
+<wire x1="18.8" y1="8.45" x2="18.6" y2="8.25" width="0.16" layer="3"/>
 <wire x1="-17.25" y1="12.1" x2="-17.145" y2="12.09" width="0" layer="19" extent="1-1"/>
 <wire x1="-6.86" y1="2.9" x2="-6.81" y2="2.85" width="0" layer="19" extent="1-1"/>
@@
 <contactref element="U$6" pad="7"/>
 <wire x1="9.38" y1="-0.14" x2="11.71" y2="-0.14" width="0.16" layer="1"/>
-<contactref element="CAN" pad="P$2"/>
-<wire x1="24.4" y1="6.5" x2="21.75" y2="6.5" width="0.16" layer="1"/>
 <wire x1="21.75" y1="6.5" x2="15.5" y2="0.25" width="0.16" layer="1"/>
 <wire x1="15.5" y1="0.25" x2="12.1" y2="0.25" width="0.16" layer="1"/>
 <wire x1="12.1" y1="0.25" x2="11.71" y2="-0.14" width="0.16" layer="1"/>
+<contactref element="U$8" pad="2"/>
+<wire x1="21.75" y1="6.5" x2="24.25" y2="6.5" width="0.16" layer="1"/>
+<wire x1="24.25" y1="6.5" x2="24.6" y2="6.45" width="0.16" layer="1"/>
 </signal>
 <signal name="CANL">
@@
 <wire x1="9.38" y1="-0.64" x2="11.81" y2="-0.64" width="0.16" layer="1"/>
 <wire x1="11.81" y1="-0.64" x2="12.2" y2="-0.25" width="0.16" layer="1"/>
-<contactref element="CAN" pad="P$1"/>
-<wire x1="24.4" y1="4" x2="19.75" y2="4" width="0.16" layer="1"/>
+<wire x1="23.85" y1="4" x2="19.75" y2="4" width="0.16" layer="1"/>
 <wire x1="19.75" y1="4" x2="15.5" y2="-0.25" width="0.16" layer="1"/>
 <wire x1="15.5" y1="-0.25" x2="12.2" y2="-0.25" width="0.16" layer="1"/>
+<contactref element="U$8" pad="1"/>
+<wire x1="23.85" y1="4" x2="24.6" y2="4.45" width="0.16" layer="1"/>
 </signal>
 <signal name="SPA">
