File: New Version/Cheetah Driver Integrated V4 connector/HKCV4.sch (EAGLE design)
At the start: 72 parts, among them Q1 TPH, Q2 TPH, Q3 TPH, Q4 TPH, Q5 TPH, Q6 TPH

Commit message: updated can connector to harwin high-reliability latching
Parts:
- removed CAN: 5267-3, con-molex-spox:5267-3
- added U$8: 3-PIN, Ben_Library:3-PIN
Connections:
- net CANH: now also U$8.P$2; no longer CAN.-2
- net CANL: now also U$8.P$1; no longer CAN.-1
- net GND: now also U$8.P$3; no longer CAN.-3
Changed lines of the file:
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@@
 <part name="PROG" library="con-jst2" deviceset="?M07B-SRSS-TB" device="S"/>
 <part name="U$9" library="Ben_Library" deviceset="XT30" device=""/>
-<part name="CAN" library="con-molex-spox" deviceset="5267-3" device=""/>
 <part name="C21" library="rcl" deviceset="C-US" device="C1206K" value="10 uF 50v"/>
 <part name="C22" library="rcl" deviceset="C-US" device="C1206K" value="10 uF 50v"/>
@@
 <part name="C28" library="rcl" deviceset="C-US" device="C1206K" value="10 uF 50v"/>
 <part name="C29" library="rcl" deviceset="C-US" device="C1206K" value="10 uF 50v"/>
+<part name="U$8" library="Ben_Library" deviceset="3-PIN" device=""/>
 </parts>
 <sheets>
@@
 <instance part="PROG" gate="-7" x="43.18" y="-43.18"/>
 <instance part="U$9" gate="G$1" x="88.9" y="-60.96"/>
-<instance part="CAN" gate="G$1" x="81.28" y="-40.64"/>
 <instance part="C21" gate="G$1" x="391.16" y="124.46"/>
 <instance part="C22" gate="G$1" x="396.24" y="124.46"/>
@@
 <instance part="C28" gate="G$1" x="421.64" y="124.46"/>
 <instance part="C29" gate="G$1" x="426.72" y="124.46"/>
+<instance part="U$8" gate="G$1" x="81.28" y="-25.4" rot="MR0"/>
 </instances>
 <busses>
@@
 </segment>
 <segment>
-<wire x1="81.28" y1="-43.18" x2="76.2" y2="-43.18" width="0.1524" layer="91"/>
+<wire x1="101.6" y1="-22.86" x2="86.36" y2="-27.94" width="0.1524" layer="91"/>
 <label x="66.04" y="-45.72" size="1.778" layer="95"/>
-<pinref part="CAN" gate="G$1" pin="-3"/>
+<pinref part="U$8" gate="G$1" pin="P$3"/>
 </segment>
 <segment>
@@
 </segment>
 <segment>
-<wire x1="81.28" y1="-40.64" x2="76.2" y2="-40.64" width="0.1524" layer="91"/>
+<wire x1="101.6" y1="-20.32" x2="86.36" y2="-25.4" width="0.1524" layer="91"/>
 <label x="68.58" y="-40.64" size="1.778" layer="95"/>
-<pinref part="CAN" gate="G$1" pin="-2"/>
+<pinref part="U$8" gate="G$1" pin="P$2"/>
 </segment>
 </net>
@@
 </segment>
 <segment>
-<wire x1="81.28" y1="-38.1" x2="76.2" y2="-38.1" width="0.1524" layer="91"/>
+<wire x1="101.6" y1="-17.78" x2="86.36" y2="-22.86" width="0.1524" layer="91"/>
 <label x="68.58" y="-38.1" size="1.778" layer="95"/>
-<pinref part="CAN" gate="G$1" pin="-1"/>
-</segment>
-</net>
+<pinref part="U$8" gate="G$1" pin="P$1"/>
+</segment>
+</net>
